File: pcb_screenshot_trial/answer.kicad_pcb (KiCad board)
At the start: 2 copper layers, 90 x 61 mm, 2 parts, among them J1 sig/gnd, J2 sig/gnd

Commit message: kkk
Parts:
- J1, J2: value sig/gnd -> SIG/GND; footprint PinHeader_1x02_P2.54mm_Vertical -> Connector_PinHeader_2.54mm:PinHeader_1x02_P2.54mm_Vertical
Routing:
- net SIG: track 86.5 -> 92.0 mm
Changed lines of the file:
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@@
 	(net 1 "SIG")
 	(net 2 "GND")
-	(footprint "PinHeader_1x02_P2.54mm_Vertical"
-		(layer "F.Cu")
-		(at 105 118)
+	(footprint "Connector_PinHeader_2.54mm:PinHeader_1x02_P2.54mm_Vertical"
+		(layer "F.Cu")
+		(at 185 118)
 		(descr "Through hole straight pin header, 1x02, 2.54mm pitch, single row")
 		(tags "Through hole pin header THT 1x02 2.54mm single row")
-		(property "Reference" "J1"
+		(property "Reference" "J2"
 			(at 0 -2.38 0)
 			(layer "F.SilkS")
@@
 			)
 		)
-		(property "Value" "sig/gnd"
+		(property "Value" "SIG/GND"
 			(at 0 4.92 0)
 			(layer "F.Fab")
@@
 		)
 	)
-	(footprint "PinHeader_1x02_P2.54mm_Vertical"
-		(layer "F.Cu")
-		(at 185 118)
+	(footprint "Connector_PinHeader_2.54mm:PinHeader_1x02_P2.54mm_Vertical"
+		(layer "F.Cu")
+		(at 105 118)
 		(descr "Through hole straight pin header, 1x02, 2.54mm pitch, single row")
 		(tags "Through hole pin header THT 1x02 2.54mm single row")
-		(property "Reference" "J2"
+		(property "Reference" "J1"
 			(at 0 -2.38 0)
 			(layer "F.SilkS")
@@
 			)
 		)
-		(property "Value" "sig/gnd"
+		(property "Value" "SIG/GND"
 			(at 0 4.92 0)
 			(layer "F.Fab")
@@
 	)
 	(gr_line
-		(start 190 151)
-		(end 100 151)
+		(start 100 90)
+		(end 190 90)
 		(stroke
 			(width 0.05)
@@
 	)
 	(gr_line
-		(start 100 90)
-		(end 190 90)
+		(start 190 151)
+		(end 100 151)
 		(stroke
 			(width 0.05)
@@
 	(segment
 		(start 142 118)
-		(end 142 112)
-		(width 0.3)
-		(layer "F.Cu")
-		(net 1)
-	)
-	(segment
-		(start 148 112)
-		(end 185 118)
-		(width 0.3)
-		(layer "F.Cu")
-		(net 1)
-	)
-	(segment
-		(start 142 112)
-		(end 148 112)
+		(end 142 124)
 		(width 0.3)
 		(layer "F.Cu")
@@
 		(width 0.3)
 		(layer "F.Cu")
+		(net 1)
+	)
+	(segment
+		(start 148 118)
+		(end 185 118)
+		(width 0.3)
+		(layer "F.Cu")
+		(net 1)
+	)
+	(segment
+		(start 142 124)
+		(end 148 124)
+		(width 0.3)
+		(layer "F.Cu")
+		(net 1)
+	)
+	(segment
+		(start 148 124)
+		(end 148 118)
+		(width 0.3)
+		(layer "F.Cu")
